File: tle5012b encoder breakout.kicad_pcb (KiCad board)
At the start: 2 copper layers, 23 x 23 mm, 12 parts, among them J1 Conn_01x02, J2 Conn_01x06, J3 Conn_01x06, U1 TLE5012

Commit message: Connected connector mounting pads to gnd plane for structural support
Parts:
- J2: value Conn_01x06 -> data-V
- J3: value Conn_01x06 -> data-H
Connections:
- J1 pad MP: (no net) -> GND
- J2 pad MP: (no net) -> GND
- J3 pad MP: (no net) -> GND
- U1 pad 1: +5V -> unconnected-(U1-Pad1)
- U1 pad 5: (no net) -> unconnected-(U1-Pad5)
- U1 pad 8: (no net) -> unconnected-(U1-Pad8)
Changed lines of the file:
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@@
   (net 7 "/H3{slash}CS")
   (net 8 "/H1{slash}SCK")
+  (net 9 "unconnected-(U1-Pad8)")
+  (net 10 "unconnected-(U1-Pad5)")
+  (net 11 "unconnected-(U1-Pad1)")
   (footprint "pkl_dipol:R_0603" (layer "F.Cu")
     (at 139 81.75 90)
@@
       (effects (font (size 1 1) (thickness 0.15)))
     )
-    (fp_text value "Conn_01x06" (at 0 4) (layer "F.Fab")
+    (fp_text value "data-V" (at 0 4) (layer "F.Fab")
       (effects (font (size 1 1) (thickness 0.15)))
     )
@@
     (pad "6" smd roundrect locked (at 3.125 1.95) (size 0.6 1.7) (layers "F.Cu" "F.Paste" "F.Mask") (roundrect_rratio 0.25)
       (net 5 "+5V") (pinfunction "Pin_6") (pintype "passive"))
-    (pad "MP" smd roundrect locked (at 4.975 -1.4) (size 1 2.8) (layers "F.Cu" "F.Paste" "F.Mask") (roundrect_rratio 0.25))
-    (pad "MP" smd roundrect locked (at -4.975 -1.4) (size 1 2.8) (layers "F.Cu" "F.Paste" "F.Mask") (roundrect_rratio 0.25))
+    (pad "MP" smd roundrect locked (at 4.975 -1.4) (size 1 2.8) (layers "F.Cu" "F.Paste" "F.Mask") (roundrect_rratio 0.25)
+      (net 2 "GND") (pinfunction "MP") (pintype "passive"))
+    (pad "MP" smd roundrect locked (at -4.975 -1.4) (size 1 2.8) (layers "F.Cu" "F.Paste" "F.Mask") (roundrect_rratio 0.25)
+      (net 2 "GND") (pinfunction "MP") (pintype "passive"))
     (model "${KISYS3DMOD}/Connector_JST.3dshapes/JST_GH_BM06B-GHS-TBT_1x06-1MP_P1.25mm_Vertical.wrl" hide
       (offset (xyz 0 0 0))
@@
     (pad "2" smd roundrect locked (at 0.625 -1.85 180) (size 0.6 1.7) (layers "F.Cu" "F.Paste" "F.Mask") (roundrect_rratio 0.25)
       (net 2 "GND") (pinfunction "Pin_2") (pintype "passive"))
-    (pad "MP" smd roundrect locked (at -2.475 1.35 180) (size 1 2.7) (layers "F.Cu" "F.Paste" "F.Mask") (roundrect_rratio 0.25))
-    (pad "MP" smd roundrect locked (at 2.475 1.35 180) (size 1 2.7) (layers "F.Cu" "F.Paste" "F.Mask") (roundrect_rratio 0.25))
+    (pad "MP" smd roundrect locked (at -2.475 1.35 180) (size 1 2.7) (layers "F.Cu" "F.Paste" "F.Mask") (roundrect_rratio 0.25)
+      (net 2 "GND") (pinfunction "MP") (pintype "passive"))
+    (pad "MP" smd roundrect locked (at 2.475 1.35 180) (size 1 2.7) (layers "F.Cu" "F.Paste" "F.Mask") (roundrect_rratio 0.25)
+      (net 2 "GND") (pinfunction "MP") (pintype "passive"))
     (model "${KISYS3DMOD}/Connector_JST.3dshapes/JST_GH_SM02B-GHS-TB_1x02-1MP_P1.25mm_Horizontal.wrl"
       (offset (xyz 0 0 0))
@@
       (effects (font (size 1 1) (thickness 0.15)))
     )
-    (fp_text value "Conn_01x06" (at 0 3.9) (layer "F.Fab")
+    (fp_text value "data-H" (at 0 3.9) (layer "F.Fab")
       (effects (font (size 1 1) (thickness 0.15)))
     )
@@
     (pad "6" smd roundrect locked (at 3.125 -1.85) (size 0.6 1.7) (layers "F.Cu" "F.Paste" "F.Mask") (roundrect_rratio 0.25)
       (net 5 "+5V") (pinfunction "Pin_6") (pintype "passive"))
-    (pad "MP" smd roundrect locked (at -4.975 1.35) (size 1 2.7) (layers "F.Cu" "F.Paste" "F.Mask") (roundrect_rratio 0.25))
-    (pad "MP" smd roundrect locked (at 4.975 1.35) (size 1 2.7) (layers "F.Cu" "F.Paste" "F.Mask") (roundrect_rratio 0.25))
+    (pad "MP" smd roundrect locked (at -4.975 1.35) (size 1 2.7) (layers "F.Cu" "F.Paste" "F.Mask") (roundrect_rratio 0.25)
+      (net 2 "GND") (pinfunction "MP") (pintype "passive"))
+    (pad "MP" smd roundrect locked (at 4.975 1.35) (size 1 2.7) (layers "F.Cu" "F.Paste" "F.Mask") (roundrect_rratio 0.25)
+      (net 2 "GND") (pinfunction "MP") (pintype "passive"))
     (model "${KISYS3DMOD}/Connector_JST.3dshapes/JST_GH_SM06B-GHS-TB_1x06-1MP_P1.25mm_Horizontal.wrl"
       (offset (xyz 0 0 0))
@@
     (fp_line (start -0.975 2.45) (end 1.95 2.45) (layer "B.Fab") (width 0.1))
     (pad "1" smd roundrect locked (at -2.575 1.905 180) (size 1.75 0.6) (layers "B.Cu" "B.Paste" "B.Mask") (roundrect_rratio 0.25)
-      (net 5 "+5V") (pinfunction "CLK/IFC") (pintype "open_collector"))
+      (net 11 "unconnected-(U1-Pad1)") (pinfunction "CLK/IFC") (pintype "open_collector"))
     (pad "2" smd roundrect locked (at -2.575 0.635 180) (size 1.75 0.6) (layers "B.Cu" "B.Paste" "B.Mask") (roundrect_rratio 0.25)
       (net 8 "/H1{slash}SCK") (pinfunction "SCK") (pintype "input"))
@@
       (net 3 "Net-(R2-Pad2)") (pinfunction "DATA") (pintype "bidirectional"))
     (pad "5" smd roundrect locked (at 2.575 -1.905 180) (size 1.75 0.6) (layers "B.Cu" "B.Paste" "B.Mask") (roundrect_rratio 0.25)
-      (pinfunction "IFA") (pintype "open_collector"))
+      (net 10 "unconnected-(U1-Pad5)") (pinfunction "IFA") (pintype "open_collector"))
     (pad "6" smd roundrect locked (at 2.575 -0.635 180) (size 1.75 0.6) (layers "B.Cu" "B.Paste" "B.Mask") (roundrect_rratio 0.25)
       (net 5 "+5V") (pinfunction "VDD") (pintype "power_in"))
@@
       (net 2 "GND") (pinfunction "GND") (pintype "power_in"))
     (pad "8" smd roundrect locked (at 2.575 1.905 180) (size 1.75 0.6) (layers "B.Cu" "B.Paste" "B.Mask") (roundrect_rratio 0.25)
-      (pinfunction "IFB") (pintype "open_collector"))
+      (net 9 "unconnected-(U1-Pad8)") (pinfunction "IFB") (pintype "open_collector"))
     (model "${KISYS3DMOD}/Package_SO.3dshapes/SO-8_3.9x4.9mm_P1.27mm.wrl"
       (offset (xyz 0 0 0))
@@
       )
     )
+  )
+  (zone (net 2) (net_name "GND") (layer "F.Cu") (hatch edge 0.508)
+    (priority 1)
+    (connect_pads yes (clearance 0.3))
+    (min_thickness 0.254) (filled_areas_thickness no)
+    (fill yes (thermal_gap 0.508) (thermal_bridge_width 0.508))
+    (polygon
+      (pts
+        (xy 141.95 76.15)
+        (xy 135 76.2)
+        (xy 135 72.55)
+        (xy 142 72.55)
+      )
+    )
+  )
+  (zone (net 2) (net_name "GND") (layer "F.Cu") (hatch edge 0.508)
+    (connect_pads yes (clearance 0.3))
+    (min_thickness 0.254) (filled_areas_thickness no)
+    (fill yes (thermal_gap 0.508) (thermal_bridge_width 0.508))
+    (polygon
+      (pts
+        (xy 144.5 92.1)
+        (xy 142.5 92.1)
+        (xy 142.5 86.7)
+        (xy 144.5 86.7)
+      )
+    )
+  )
+  (zone (net 2) (net_name "GND") (layer "F.Cu") (hatch edge 0.508)
+    (connect_pads yes (clearance 0.3))
+    (min_thickness 0.254) (filled_areas_thickness no)
+    (fill yes (thermal_gap 0.508) (thermal_bridge_width 0.508))
+    (polygon
+      (pts
+        (xy 134.5 92.1)
+        (xy 132.5 92.1)
+        (xy 132.5 86.7)
+        (xy 134.5 86.7)
+      )
+    )
